Commit message: change to base scan

File: robot_bringup/urdf/mecanum_drive.xacro.urdf (robot description, URDF)
Before this commit: robot mecanum_vehicle, 8 links, 7 joints
Links:
- removed link laser_frame
- added link base_scan, mass 0.01; visual mesh filename=file://$(find robot_bringup)/meshes/VLP16/VLP16_scan.dae
Joints:
- joint velodyne_base_scan_joint: child laser_frame -> base_scan
